Commit message: Imported upstream version '0.4.3' of 'upstream'

File: magni_description/urdf/magni.urdf.xacro (robot description, xacro)
@@ -76,5 +76,5 @@
   <xacro:if value="${raspicam_mount == 'upward'}">
     <xacro:raspicam>
-      <origin xyz="0.035 0.15 0.14" rpy="0 0 -1.5707"/>
+      <origin xyz="0.035 0.15 0.14" rpy="0 0 ${pi}"/>
     </xacro:raspicam>
   </xacro:if>

Commit message: Imported upstream version '0.5.0' of 'upstream'

File: magni_description/urdf/magni.urdf.xacro (robot description, xacro)
@@ -1,81 +1,157 @@
 <?xml version="1.0"?>
-<robot xmlns:xacro="http://www.ros.org/wiki/xacro" name="magni">
-  <xacro:arg name="raspicam_mount" default="forward"/>
-  <xacro:property name="raspicam_mount" value="$(arg raspicam_mount)"/>
+<robot xmlns:xacro="http://wiki.ros.org/xacro" name="magni">
   <xacro:arg name="sonars_installed" default="true"/>
   <xacro:property name="sonars_installed" value="$(arg sonars_installed)"/>
-  <!-- base links for the urdf -->
-  <link name="base_link"/>
+  <xacro:arg name="camera_extrinsics_file" default=""/>
+  <xacro:property name="camera_extrinsics_file" value="$(arg camera_extrinsics_file)"/>
+  <xacro:arg name="lidar_extrinsics_file" default=""/>
+  <xacro:property name="lidar_extrinsics_file" value="$(arg lidar_extrinsics_file)"/>
+  <xacro:property name="wheel_r" value="0.1" />
+  <xacro:property name="wheel_xpos" value="0.11" />
+  <xacro:include filename="$(find magni_description)/urdf/magni.transmission.xacro" />
+  <xacro:include filename="$(find magni_description)/urdf/magni.gazebo.xacro" />
+  <xacro:include filename="$(find magni_description)/urdf/inertial.xacro" />
+  <xacro:include filename="$(find magni_description)/urdf/sensors/sonar_hc-sr04.xacro" />
+  <xacro:include filename="$(find magni_description)/urdf/sensors/raspi_camera.xacro" />
+  <xacro:include filename="$(find magni_description)/urdf/sensors/hokuyo_lidar.xacro" />
+  <!-- Robot base_link -->
+  <link name="base_link">
+    <visual>
+      <origin xyz="${-wheel_xpos} 0 ${-wheel_r+0.071}" rpy="0 0 0" />
+      <geometry>
+        <mesh filename="package://magni_description/meshes/magni_body.dae" />
+      </geometry>
+    </visual>
+	<visual>
+      <origin xyz="${-wheel_xpos-0.169} 0.17 ${-wheel_r+0.09}" rpy="0 0 ${pi}" />
+      <geometry>
+        <mesh filename="package://magni_description/meshes/caster_wheel.dae" />
+      </geometry>
+    </visual>
+	<visual>
+      <origin xyz="${-wheel_xpos-0.169} -0.17 ${-wheel_r+0.09}" rpy="0 0 ${pi}" />
+      <geometry>
+        <mesh filename="package://magni_description/meshes/caster_wheel.dae" />
+      </geometry>
+    </visual>
+    <collision>
+	  <origin xyz="${-wheel_xpos} 0 ${-wheel_r+0.151}" rpy="0 0 0" />
+      <geometry>
+        <box size="0.398 0.268 0.160"/>
+      </geometry>
+    </collision>
+    <collision>
+      <origin xyz="${-wheel_xpos-0.026} 0 ${-wheel_r+0.248}" rpy="0 0 0" />
+      <geometry>
+        <box size="0.375 0.268 0.034"/>
+      </geometry>
+    </collision>
+    <collision>
+      <origin xyz="${-wheel_xpos-0.169} 0.169 ${-wheel_r+0.106}" rpy="0 0 0" />
+      <geometry>
+        <box size="0.1 0.07 0.07"/>
+      </geometry>
+    </collision>
+    <collision>
+      <origin xyz="${-wheel_xpos-0.169} -0.169 ${-wheel_r+0.106}" rpy="0 0 0" />
+      <geometry>
+        <box size="0.1 0.07 0.07"/>
+      </geometry>
+    </collision>
+    <xacro:box_inertial_with_origin  x="0.398" y="0.221" z="0.150" mass="10.0">
+      <origin xyz="-0.15 0 0.03" rpy="0 0 0" />
+    </xacro:box_inertial_with_origin>
+  </link>
+  <!-- Fixed offset from the floor to the center of the wheels -->
   <link name="base_footprint"/>
-  <!-- Fixed offset from the floor to the center of the wheels -->
   <joint name="base_footprint_joint" type="fixed">
-    <parent link="base_link"/>
-    <child link="base_footprint"/>
-    <origin xyz="0 0 -0.1" rpy="0 0 0"/>
+    <parent link="base_footprint"/>
+    <child link="base_link"/>
+    <origin xyz="0 0 ${wheel_r}" rpy="0 0 0"/>
   </joint>
   <!-- Macro for defining wheels -->
-  <xacro:macro name="wheel" params="name">
-    <link name="${name}_wheel"/>
-    <joint name="${name}_wheel_joint" type="continuous">
+  <xacro:macro name="wheel" params="prefix reflect">
+    <link name="${prefix}_wheel">
+      <visual>
+        <origin xyz="${-0.071*reflect} 0 0" rpy="0 ${(reflect-1)*pi/2} 0" />
+        <geometry>
+          <mesh filename="package://magni_description/meshes/front_wheel.dae" />
+        </geometry>
+      </visual>
+      <collision>
+        <origin xyz="0 0 0" rpy="0 ${pi/2} 0" />
+        <geometry>
+          <cylinder radius="${wheel_r}" length="0.05"/>
+        </geometry>
+      </collision>
+      <collision>
+        <origin xyz="${0.033*reflect} 0 0" rpy="0 ${pi/2} 0" />
+        <geometry>
+          <cylinder radius="0.064" length="0.016"/>
+        </geometry>
+      </collision>
+      <xacro:cylinder_inertial_with_origin radius="${wheel_r}" length="0.05" mass="3.34">
+        <origin xyz="0 0 0" rpy="0 ${pi/2} 0" />
+      </xacro:cylinder_inertial_with_origin>
+    </link>
+    <joint name="${prefix}_wheel_joint" type="continuous">
+      <axis xyz="1 0 0" rpy="0 0 0" />
       <parent link="base_link"/>
-      <child link="${name}_wheel"/>
-      <xacro:if value="${name == 'left'}">
-        <origin xyz="0 0.165 0" rpy="0 0 0" />
-        <axis xyz="0 1 0" />
-      </xacro:if>
-      <xacro:if value="${name == 'right'}">
-        <origin xyz="0 -0.165 0" rpy="${pi} 0 0" />
-        <axis xyz="0 -1 0" />
-      </xacro:if>
+      <child link="${prefix}_wheel"/>
+      <origin xyz="0 ${0.163*reflect} 0" rpy="0 0 ${pi/2}"/>
     </joint>
   </xacro:macro>
-  <xacro:wheel name="left"/>
-  <xacro:wheel name="right"/>
-  <!-- Macro for defining sonars -->
-  <xacro:macro name="sonar" params="name *origin">
-    <link name="${name}"/>
-    <joint name="${name}" type="fixed">
+  <xacro:wheel prefix="left" reflect="1"/>
+  <xacro:wheel prefix="right" reflect="-1"/>
+  <!-- Macro for defining caster wheels -->
+  <xacro:macro name="caster_wheel" params="prefix reflect">
+    <link name="${prefix}_caster_wheel">
+      <collision>
+        <origin xyz="${-wheel_xpos-0.19} ${reflect*0.169} ${-wheel_r+0.04}" rpy="0 0 0" />
+        <geometry>
+          <sphere radius="0.04"/>
+        </geometry>
+      </collision>
+    </link>
+    <joint name="${prefix}_caster_wheel_joint" type="fixed">
       <parent link="base_link"/>
-      <child link="${name}"/>
-      <xacro:insert_block name="origin"/>
+      <child link="${prefix}_caster_wheel"/>
     </joint>
   </xacro:macro>
+  <xacro:caster_wheel prefix="left" reflect="1"/>
+  <xacro:caster_wheel prefix="right" reflect="-1"/>
   <!-- Define all sonars, if sonars_installed set to 1 -->
   <xacro:if value="${sonars_installed}">
-    <xacro:sonar name="sonar_0">
+    <xacro:sonar_hc-sr04 name="sonar_0" connected_to="base_link">
       <origin xyz="0.01 -0.14 0.15" rpy="0 0 ${-pi/2}"/>
-    </xacro:sonar>
-    <xacro:sonar name="sonar_1">
+    </xacro:sonar_hc-sr04>
+    <xacro:sonar_hc-sr04 name="sonar_1" connected_to="base_link">
       <origin xyz="0.08 -0.07 0.15" rpy="0 0 0.785"/>
-    </xacro:sonar>
-    <xacro:sonar name="sonar_2">
+    </xacro:sonar_hc-sr04>
+    <xacro:sonar_hc-sr04 name="sonar_2" connected_to="base_link">
       <origin xyz="0.08 -0.01 0.15" rpy="0 0 -0.785"/>
-    </xacro:sonar>
-    <xacro:sonar name="sonar_3">
+    </xacro:sonar_hc-sr04>
+    <xacro:sonar_hc-sr04 name="sonar_3" connected_to="base_link">
       <origin xyz="0.08 0.04 0.15" rpy="0 0 0"/>
-    </xacro:sonar>
-    <xacro:sonar name="sonar_4">
+    </xacro:sonar_hc-sr04>
+    <xacro:sonar_hc-sr04 name="sonar_4" connected_to="base_link">
       <origin xyz="0.01 0.14 0.15" rpy="0 0 ${pi/2}"/>
-    </xacro:sonar>
+    </xacro:sonar_hc-sr04>
   </xacro:if>
-  <!-- Macro for defining raspicam -->
-  <xacro:macro name="raspicam" params="*origin">
-    <link name="raspicam"/>
-    <joint name="raspicam" type="fixed">
-      <parent link="base_link"/>
-      <child link="raspicam"/>
-      <xacro:insert_block name="origin"/>
-    </joint>
-  </xacro:macro>
-  <!-- Define raspicam based on the raspicam_mount argument -->
-  <xacro:if value="${raspicam_mount == 'forward'}">
-    <xacro:raspicam>
-      <origin xyz="0.035 0.085 0.14" rpy="1.15191731 0 1.5707"/>
-    </xacro:raspicam>
+  <!-- Define camera -->
+  <xacro:if value="${camera_extrinsics_file != ''}">
+    <xacro:property name="cam_extrinsics" value="${load_yaml(camera_extrinsics_file)}"/>
+    <xacro:raspi_camera name="raspicam" connected_to="base_link">
+      <origin xyz="${cam_extrinsics['x']} ${cam_extrinsics['y']} ${cam_extrinsics['z']}"
+        rpy="${cam_extrinsics['roll']} ${cam_extrinsics['pitch']} ${cam_extrinsics['yaw']}"/>
+    </xacro:raspi_camera>
   </xacro:if>
-  <xacro:if value="${raspicam_mount == 'upward'}">
-    <xacro:raspicam>
-      <origin xyz="0.035 0.15 0.14" rpy="0 0 ${pi}"/>
-    </xacro:raspicam>
+  <!-- Define Lidar -->
+  <xacro:if value="${lidar_extrinsics_file != ''}">
+    <xacro:property name="lidar_extrinsics" value="${load_yaml(lidar_extrinsics_file)}"/>
+    <xacro:hokuyo_lidar name="laser" connected_to="base_link">
+      <origin xyz="${lidar_extrinsics['x']} ${lidar_extrinsics['y']} ${lidar_extrinsics['z']}"
+        rpy="${lidar_extrinsics['roll']} ${lidar_extrinsics['pitch']} ${lidar_extrinsics['yaw']}"/>
+    </xacro:hokuyo_lidar>
   </xacro:if>
 </robot>
